File: SI_kicad.sch (KiCad schematic (older format))
At the start: 88 parts, among them J1 Conn_01x16_Female, J2 SCW_TERM_01x02, J3 Conn_02x05_Counter_Clockwise, J4 Conn_01x05_Male, J5 Conn_01x05_Female, J6 Conn_01x02, J7 Conn_01x02, Q1 BC549, Q2 BC557C, Q3 IRL7833, SW1 SW_Push, U1 STM32F103C8Tx, U2 AMS1117-3.3, U3 TPS5430DDA, U4 LM358, Y1 8M

Commit message: 1.1
Parts:
- C16: value 15p -> 10n
- C18: value 100n -> 2u
- C2, C3: value 22n -> 22p
- R16: value 15k -> 10k
- R17: value 33k -> 3.3k
- R4, R5: value 220R -> 10k
- R6: value 15k -> 16k
- R7: value 5k -> 1.6k
- RV1: value 1K -> 10K
Other:
- note added: "3.27V"
Changed lines of the file:
@@
 P 7150 1450
 F 0 "R7" H 7220 1496 50  0000 L CNN
-F 1 "5k" H 7220 1405 50  0000 L CNN
+F 1 "1.6k" H 7220 1405 50  0000 L CNN
 F 2 "Resistor_SMD:R_0805_2012Metric_Pad1.15x1.40mm_HandSolder" V 7080 1450 50  0001 C CNN
 F 3 "~" H 7150 1450 50  0001 C CNN
@@
 P 7150 1050
 F 0 "R6" H 7220 1096 50  0000 L CNN
-F 1 "15k" H 7220 1005 50  0000 L CNN
+F 1 "16k" H 7220 1005 50  0000 L CNN
 F 2 "Resistor_SMD:R_0805_2012Metric_Pad1.15x1.40mm_HandSolder" V 7080 1050 50  0001 C CNN
 F 3 "~" H 7150 1050 50  0001 C CNN
@@
 P 8550 850
 F 0 "C16" V 8800 850 50  0000 L CNN
-F 1 "15p" V 8700 900 50  0000 L CNN
+F 1 "10n" V 8700 900 50  0000 L CNN
 F 2 "Capacitor_SMD:C_0805_2012Metric_Pad1.15x1.40mm_HandSolder" H 8588 700 50  0001 C CNN
 F 3 "~" H 8550 850 50  0001 C CNN
@@
 P 9950 1050
 F 0 "C18" H 10100 1050 50  0000 L CNN
-F 1 "100n" H 10100 1150 50  0000 L CNN
+F 1 "2u" H 10100 1150 50  0000 L CNN
 F 2 "Capacitor_SMD:C_0805_2012Metric_Pad1.15x1.40mm_HandSolder" H 9988 900 50  0001 C CNN
 F 3 "~" H 9950 1050 50  0001 C CNN
@@
 P 10450 1000
 F 0 "R16" H 10550 1050 50  0000 L CNN
-F 1 "15k" H 10520 955 50  0000 L CNN
+F 1 "10k" H 10520 955 50  0000 L CNN
 F 2 "Resistor_SMD:R_0805_2012Metric_Pad1.15x1.40mm_HandSolder" V 10380 1000 50  0001 C CNN
 F 3 "~" H 10450 1000 50  0001 C CNN
@@
 P 10450 1450
 F 0 "R17" H 10520 1496 50  0000 L CNN
-F 1 "33k" H 10520 1405 50  0000 L CNN
+F 1 "3.3k" H 10520 1405 50  0000 L CNN
 F 2 "Resistor_SMD:R_0805_2012Metric_Pad1.15x1.40mm_HandSolder" V 10380 1450 50  0001 C CNN
 F 3 "~" H 10450 1450 50  0001 C CNN
@@
 P 900 2400
 F 0 "C3" V 1050 2350 50  0000 L CNN
-F 1 "22n" V 750 2350 50  0000 L CNN
+F 1 "22p" V 750 2350 50  0000 L CNN
 F 2 "Capacitor_SMD:C_0805_2012Metric_Pad1.15x1.40mm_HandSolder" H 938 2250 50  0001 C CNN
 F 3 "~" H 900 2400 50  0001 C CNN
@@
 P 900 2050
 F 0 "C2" V 1150 2000 50  0000 L CNN
-F 1 "22n" V 1050 2000 50  0000 L CNN
+F 1 "22p" V 1050 2000 50  0000 L CNN
 F 2 "Capacitor_SMD:C_0805_2012Metric_Pad1.15x1.40mm_HandSolder" H 938 1900 50  0001 C CNN
 F 3 "~" H 900 2050 50  0001 C CNN
@@
 P 3100 7350
 F 0 "RV1" H 2950 7400 50  0000 C CNN
-F 1 "1K" H 2950 7300 50  0000 C CNN
+F 1 "10K" H 2950 7300 50  0000 C CNN
 F 2 "Potentiometer_THT:Potentiometer_Bourns_3296W_Vertical" H 3100 7350 50  0001 C CNN
 F 3 "~" H 3100 7350 50  0001 C CNN
@@
 P 6600 5600
 F 0 "R4" V 6807 5600 50  0000 C CNN
-F 1 "220R" V 6716 5600 50  0000 C CNN
+F 1 "10k" V 6716 5600 50  0000 C CNN
 F 2 "Resistor_SMD:R_0805_2012Metric_Pad1.15x1.40mm_HandSolder" V 6530 5600 50  0001 C CNN
 F 3 "~" H 6600 5600 50  0001 C CNN
@@
 P 6600 6050
 F 0 "R5" V 6807 6050 50  0000 C CNN
-F 1 "220R" V 6716 6050 50  0000 C CNN
+F 1 "10k" V 6716 6050 50  0000 C CNN
 F 2 "Resistor_SMD:R_0805_2012Metric_Pad1.15x1.40mm_HandSolder" V 6530 6050 50  0001 C CNN
 F 3 "~" H 6600 6050 50  0001 C CNN
@@
 	1    0    0    -1
 $EndComp
+Text Notes 7150 1350 0    50   ~ 0
+3.27V
 $EndSCHEMATC
