File: SI_kicad.kicad_sch (KiCad schematic)
At the start: 88 parts, among them J1 Conn_01x16_Female, J2 SCW_TERM_01x02, J3 Conn_02x05_Counter_Clockwise, J4 Conn_01x05_Male, J5 Conn_01x05_Female, J6 Conn_01x02, J7 Conn_01x02, Q1 BC549, Q2 BC557C, Q3 IRL7833, SW1 SW_Push, U1 STM32F103C8Tx, U2 AMS1117-3.3, U3 TPS5430DDA, U4 LM358, Y1 8M

Commit message: 2.0
Parts:
- removed BZ1: Buzzer, Buzzer_Beeper:Buzzer_12x9.5RM7.6, symbol Device:Buzzer
- removed C1, C11, C13, C15, C17, C19, C21, C6, C7: 100n, Capacitor_SMD:C_0805_2012Metric_Pad1.15x1.40mm_HandSolder, symbol Device:C
- removed C10, C12, C14, C16, C20, C4, C5: 10n, Capacitor_SMD:C_0805_2012Metric_Pad1.15x1.40mm_HandSolder, symbol Device:C
- removed C18: 2u, Capacitor_SMD:C_0805_2012Metric_Pad1.15x1.40mm_HandSolder, symbol Device:C
- removed C2, C3: 22p, Capacitor_SMD:C_0805_2012Metric_Pad1.15x1.40mm_HandSolder, symbol Device:C
- removed C8: 4.7u, Capacitor_THT:CP_Radial_D5.0mm_P2.50mm, symbol SI_kicad-rescue:CP-Device
- removed C9: 100u, Capacitor_THT:CP_Radial_D6.3mm_P2.50mm, symbol SI_kicad-rescue:CP-Device
- removed D1: LED, LED_SMD:LED_0805_2012Metric_Pad1.15x1.40mm_HandSolder, symbol Device:LED
- removed D2: VS-KBPC806, Diode_THT:Diode_Bridge_Vishay_KBPC6, symbol Diode_Bridge:VS-KBPC806
- removed D3, D4: 1N4001, Diode_THT:D_DO-41_SOD81_P10.16mm_Horizontal, symbol Diode:1N4001
- removed F1: 3A, Fuse:Fuseholder_Cylinder-5x20mm_Schurter_0031_8201_Horizontal_Open, symbol Device:Fuse
- removed H1, H2, H3, H4, H5, H6, H7, H8: MountingHole, MountingHole:MountingHole_2.7mm_M2.5_DIN965_Pad, symbol Mechanical:MountingHole
- removed H9: Logo_Open_Hardware_Small, Symbol:OSHW-Logo_5.7x6mm_Copper, symbol Graphic:Logo_Open_Hardware_Small
- removed J1: Conn_01x16_Female, Connector_PinSocket_2.54mm:PinSocket_1x16_P2.54mm_Vertical, symbol Connector:Conn_01x16_Female
- removed J2: SCW_TERM_01x02, TerminalBlock:TerminalBlock_Altech_AK300-2_P5.00mm, symbol Connector:Screw_Terminal_01x02
- removed J3: Conn_02x05_Counter_Clockwise, Connector_PinHeader_2.54mm:PinHeader_2x05_P2.54mm_Vertical, symbol Connector_Generic:Conn_02x05_Counter_Clockwise
- removed J4: Conn_01x05_Male, Connector_PinHeader_2.54mm:PinHeader_1x05_P2.54mm_Horizontal, symbol Connector:Conn_01x05_Male
- removed J5: Conn_01x05_Female, Connector_PinSocket_2.54mm:PinSocket_1x05_P2.54mm_Vertical, symbol Connector:Conn_01x05_Female
- removed J6, J7: Conn_01x02, Connector_PinHeader_2.54mm:PinHeader_1x02_P2.54mm_Vertical, symbol Connector_Generic:Conn_01x02
- removed L1, L2: INDUCTOR, Inductor_SMD:L_Coilcraft_LPS5030, symbol pspice:INDUCTOR
- removed L3: INDUCTOR, Inductor_THT:L_Axial_L5.3mm_D2.2mm_P7.62mm_Horizontal_Vishay_IM-1, symbol pspice:INDUCTOR
- removed NT1, NT2: Net-Tie_2, NetTie:NetTie-2_SMD_Pad0.5mm, symbol SI_kicad-rescue:Net-Tie_2-Device
- removed Q1: BC549, Package_TO_SOT_THT:TO-92, symbol Device:Q_NPN_CBE
- removed Q2: BC557C, Package_TO_SOT_THT:TO-92, symbol Device:Q_PNP_CBE
- removed Q3: IRL7833, Package_TO_SOT_THT:TO-220-3_Vertical, symbol Transistor_FET:IRF3205
- removed R1, R10, R16, R4, R5: 10k, Resistor_SMD:R_0805_2012Metric_Pad1.15x1.40mm_HandSolder, symbol Device:R
- removed R11, R14, R9: 100k, Resistor_SMD:R_0805_2012Metric_Pad1.15x1.40mm_HandSolder, symbol Device:R
- removed R12: 1k, Resistor_SMD:R_0805_2012Metric_Pad1.15x1.40mm_HandSolder, symbol Device:R
- removed R13: R, Resistor_SMD:R_0805_2012Metric_Pad1.15x1.40mm_HandSolder, symbol Device:R
- removed R15: 470R, Resistor_SMD:R_0805_2012Metric_Pad1.15x1.40mm_HandSolder, symbol Device:R
- removed R17: 3.3k, Resistor_SMD:R_0805_2012Metric_Pad1.15x1.40mm_HandSolder, symbol Device:R
- removed R2: 220R, Resistor_SMD:R_0805_2012Metric_Pad1.15x1.40mm_HandSolder, symbol Device:R
- removed R3, R8: 100R, Resistor_SMD:R_0805_2012Metric_Pad1.15x1.40mm_HandSolder, symbol Device:R
- removed R6: 16k, Resistor_SMD:R_0805_2012Metric_Pad1.15x1.40mm_HandSolder, symbol Device:R
- removed R7: 1.6k, Resistor_SMD:R_0805_2012Metric_Pad1.15x1.40mm_HandSolder, symbol Device:R
- removed RV1: 10K, Potentiometer_THT:Potentiometer_Bourns_3296W_Vertical, symbol SI_kicad-rescue:R_POT-Device
- removed RV2: 500k, Potentiometer_THT:Potentiometer_Bourns_3296W_Vertical, symbol SI_kicad-rescue:R_POT-Device
- removed RV3: 50k, Potentiometer_THT:Potentiometer_Bourns_3296W_Vertical, symbol SI_kicad-rescue:R_POT-Device
- removed SW1: SW_Push, Button_Switch_SMD:SW_SPST_EVQPE1, symbol Switch:SW_Push
- removed TP1, TP10, TP11, TP2, TP3, TP4, TP5, TP6, TP7, TP8, TP9: TestPoint, TestPoint:TestPoint_Pad_D2.0mm, symbol Connector:TestPoint
- removed U1: STM32F103C8Tx, Package_QFP:LQFP-48_7x7mm_P0.5mm, symbol MCU_ST_STM32F1:STM32F103C8Tx
- removed U2: AMS1117-3.3, Package_TO_SOT_SMD:SOT-223, symbol Regulator_Linear:AMS1117-3.3
- removed U3: TPS5430DDA, Package_SO:TI_SO-PowerPAD-8_ThermalVias, symbol Regulator_Switching:TPS5430DDA
- removed U4: LM358, Package_SO:SO-8_3.9x4.9mm_P1.27mm, symbol Amplifier_Operational:LM358
- removed Y1: 8M, Crystal:Resonator-2Pin_W10.0mm_H5.0mm, symbol Device:Crystal
Connections:
- no-connect marks 23 -> 0
Other:
- added sheet Analog (Analog.kicad_sch)
- added sheet Power (Power.kicad_sch)
- added sheet uC (uc.kicad_sch)
- note removed: "3.27V"
